File: InteractiveGuitar.kicad_pcb (KiCad board)
At the start: 2 copper layers, 54 x 60 mm, 44 parts, among them J1 Conn_02x06_Odd_Even, J2 Conn_01x03, J3 Conn_02x06_Odd_Even, J4 Conn_01x10, J5 Conn_01x10, J6 Conn_01x03, J7 Conn_01x02, J8 Conn_01x05, U1 ADXL337BCPZ–RL, U2 MAX4466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

Commit message: changed connection bits
Parts:
- added mouse-bite-2mm-slot: VAL**, Panelization:mouse-bite-2mm-slot, F.Cu at (165.4, 101.0)
- added mouse-bite-2mm-slot: VAL**, Panelization:mouse-bite-2mm-slot, F.Cu at (128.5, 101.0)
- moved mouse-bite-2mm-slot 0.36 mm to (147.0, 101.0)
Other:
- outline, holes or cut-outs redrawn

Commit message: fixed mic polarity
Parts:
- MIC1: footprint digikey-footprints:Mic_CMA-4544PF-W -> Adafruit MAX4466 Mic Amp:ELECTRET_9.7
- turned MIC1 to 90 degrees
Routing:
- net AGND: track 24.2 -> 28.8 mm
