File: Sensors.sch (KiCad schematic (older format))
At the start: 32 parts, among them J1 Conn_02x06_Odd_Even, J2 Conn_01x03, U1 ADXL337BCPZ–RL, U2 MAX4466\"\"

Commit message: fixed mic polarity
Parts:
- MIC1: footprint digikey-footprints:Mic_CMA-4544PF-W -> Adafruit MAX4466 Mic Amp:ELECTRET_9.7
